Commit message: [hydragon]merge collision conflict solution, and modify each link's inertia

File: robots/hydragon/urdf/common.xacro (robot description, xacro)
@@ -5,5 +5,6 @@
       <origin xyz="-0.056027 -0.0013733 0.0074745" rpy="0.0 -0.0 0.0"/>
       <mass value="0.42744"/>
-      <inertia ixx="0.00021055" ixy="3.1246e-10" ixz="-4.0813e-08" iyy="0.00010191" iyz="-4.0104e-07" izz="0.00021817"/>
+      <!-- <inertia ixx="0.00021055" ixy="3.1246e-10" ixz="-4.0813e-08" iyy="0.00010191" iyz="-4.0104e-07" izz="0.00021817"/> -->
+      <inertia ixx="6.32212e-04" ixy="4.40e-07" ixz="8.6305e-05" iyy="7.27448e-04" iyz="-1.4140e-05" izz="4.34901e-04"/>
     </inertial>
     <visual>
@@ -30,5 +31,6 @@
       <origin xyz="-0.16731 0.025056 -0.00016724" rpy="0.0 -0.0 0.0"/>
       <mass value="0.36482"/>
-      <inertia ixx="0.00016623" ixy="-3.3215e-07" ixz="-5.731e-09" iyy="0.00018621" iyz="-6.8029e-09" izz="0.00025293"/>
+      <!-- <inertia ixx="0.00016623" ixy="-3.3215e-07" ixz="-5.731e-09" iyy="0.00018621" iyz="-6.8029e-09" izz="0.00025293"/> -->
+      <inertia ixx="4.377329e-03" ixy="8.6412e-05" ixz="1.1901e-07" iyy="5.095606e-03" iyz="1.335e-06" izz="9.365966e-03"/>
     </inertial>
     <visual>
@@ -83,5 +85,6 @@
       <origin xyz="-3.541e-05 0.00191 0.0014323" rpy="0.0 -0.0 0.0"/>
       <mass value="0.32337"/>
-      <inertia ixx="0.0012194" ixy="2.2289e-07" ixz="-1.5989e-07" iyy="0.00099811" iyz="1.3306e-05" izz="0.0019906"/>
+      <!-- <inertia ixx="0.0012194" ixy="2.2289e-07" ixz="-1.5989e-07" iyy="0.00099811" iyz="1.3306e-05" izz="0.0019906"/> -->
+      <inertia ixx="2.041188e-03" ixy="-2.45e-07" ixz="3.31e-07" iyy="1.024308e-03" iyz="-1.287e-06" izz="2.793384e-03"/>
     </inertial>
     <visual>
@@ -93,8 +96,13 @@
   </link>
   <link name="thrust1">
-    <inertial>
-      <origin xyz="-2.7492e-06 -2.3311e-06 0.0039586" rpy="0.0 -0.0 0.0"/>
-      <mass value="0.010724"/>
-      <inertia ixx="1.6559e-05" ixy="-1.3587e-09" ixz="-2.9948e-11" iyy="1.6561e-05" iyz="1.3019e-11" izz="3.3082e-05"/>
+    <!-- <inertial> -->
+    <!--   <origin xyz="-2.7492e-06 -2.3311e-06 0.0039586" rpy="0.0 -0.0 0.0"/> -->
+    <!--   <mass value="0.010724"/> -->
+    <!--   <inertia ixx="1.6559e-05" ixy="-1.3587e-09" ixz="-2.9948e-11" iyy="1.6561e-05" iyz="1.3019e-11" izz="3.3082e-05"/> -->
+    <!-- </inertial> -->
+    <inertial>
+      <origin xyz="0 0 0" rpy="0 0 0"/>
+      <mass value="0.0001"/>
+      <inertia ixx="0.00001" ixy="0.0" ixz="0.0" iyy="0.00001" iyz="0.0" izz="0.00002"/>
     </inertial>
     <visual>
@@ -116,5 +124,6 @@
       <origin xyz="-0.036672 -2.1161e-05 0.0081671" rpy="0.0 -0.0 0.0"/>
       <mass value="0.31592"/>
-      <inertia ixx="5.7571e-05" ixy="6.2131e-09" ixz="8.7034e-08" iyy="9.2786e-05" iyz="-8.9098e-12" izz="7.7319e-05"/>
+      <!-- <inertia ixx="5.7571e-05" ixy="6.2131e-09" ixz="8.7034e-08" iyy="9.2786e-05" iyz="-8.9098e-12" izz="7.7319e-05"/> -->
+      <inertia ixx="4.69603e-04" ixy="1.87e-07" ixz="-3.7323e-05" iyy="5.56006e-04" iyz="-2.016e-05" izz="1.49828e-04"/>
     </inertial>
     <visual>
@@ -141,5 +150,6 @@
       <origin xyz="-0.056027 -0.0013733 0.0074745" rpy="0.0 -0.0 0.0"/>
       <mass value="0.42744"/>
-      <inertia ixx="0.00021055" ixy="3.1247e-10" ixz="-4.0813e-08" iyy="0.00010191" iyz="-4.0104e-07" izz="0.00021817"/>
+      <!-- <inertia ixx="0.00021055" ixy="3.1247e-10" ixz="-4.0813e-08" iyy="0.00010191" iyz="-4.0104e-07" izz="0.00021817"/> -->
+      <inertia ixx="6.32212e-04" ixy="4.40e-07" ixz="8.6305e-05" iyy="7.27448e-04" iyz="-1.4140e-05" izz="4.34901e-04"/>
     </inertial>
     <visual>
@@ -166,5 +176,6 @@
       <origin xyz="-0.16731 0.025056 -0.00016724" rpy="0.0 -0.0 0.0"/>
       <mass value="0.36482"/>
-      <inertia ixx="0.00016623" ixy="-3.3215e-07" ixz="-5.731e-09" iyy="0.00018621" iyz="-6.8029e-09" izz="0.00025293"/>
+      <!-- <inertia ixx="0.00016623" ixy="-3.3215e-07" ixz="-5.731e-09" iyy="0.00018621" iyz="-6.8029e-09" izz="0.00025293"/> -->
+      <inertia ixx="4.377329e-03" ixy="8.6412e-05" ixz="1.1901e-07" iyy="5.095606e-03" iyz="1.335e-06" izz="9.365966e-03"/>
     </inertial>
     <visual>
@@ -221,5 +232,6 @@
       <origin xyz="-3.541e-05 0.00191 0.0014323" rpy="0.0 -0.0 0.0"/>
       <mass value="0.32337"/>
-      <inertia ixx="0.0012194" ixy="2.2289e-07" ixz="-1.5989e-07" iyy="0.00099811" iyz="1.3306e-05" izz="0.0019906"/>
+      <!-- <inertia ixx="0.0012194" ixy="2.2289e-07" ixz="-1.5989e-07" iyy="0.00099811" iyz="1.3306e-05" izz="0.0019906"/> -->
+      <inertia ixx="2.041188e-03" ixy="-2.45e-07" ixz="3.31e-07" iyy="1.024308e-03" iyz="-1.287e-06" izz="2.793384e-03"/>
     </inertial>
     <visual>
@@ -231,8 +243,13 @@
   </link>
   <link name="thrust2">
-    <inertial>
-      <origin xyz="-2.5539e-06 -2.3067e-06 0.0039586" rpy="0.0 -0.0 0.0"/>
-      <mass value="0.010724"/>
-      <inertia ixx="1.6559e-05" ixy="-1.2942e-09" ixz="-2.6675e-11" iyy="1.6561e-05" iyz="1.4693e-11" izz="3.3081e-05"/>
+    <!-- <inertial> -->
+    <!--   <origin xyz="-2.5539e-06 -2.3067e-06 0.0039586" rpy="0.0 -0.0 0.0"/> -->
+    <!--   <mass value="0.010724"/> -->
+    <!--   <inertia ixx="1.6559e-05" ixy="-1.2942e-09" ixz="-2.6675e-11" iyy="1.6561e-05" iyz="1.4693e-11" izz="3.3081e-05"/> -->
+    <!-- </inertial> -->
+    <inertial>
+      <origin xyz="0 0 0" rpy="0 0 0"/>
+      <mass value="0.0001"/>
+      <inertia ixx="0.00001" ixy="0.0" ixz="0.0" iyy="0.00001" iyz="0.0" izz="0.00002"/>
     </inertial>
     <visual>
@@ -254,5 +271,6 @@
       <origin xyz="-0.036672 -2.1161e-05 0.0081671" rpy="0.0 -0.0 0.0"/>
       <mass value="0.31592"/>
-      <inertia ixx="5.7571e-05" ixy="6.2131e-09" ixz="8.7034e-08" iyy="9.2786e-05" iyz="-8.9132e-12" izz="7.7319e-05"/>
+      <!-- <inertia ixx="5.7571e-05" ixy="6.2131e-09" ixz="8.7034e-08" iyy="9.2786e-05" iyz="-8.9132e-12" izz="7.7319e-05"/> -->
+      <inertia ixx="4.69603e-04" ixy="1.87e-07" ixz="-3.7323e-05" iyy="5.56006e-04" iyz="-2.016e-05" izz="1.49828e-04"/>
     </inertial>
     <visual>
@@ -279,5 +297,6 @@
       <origin xyz="-0.056027 -0.0013733 0.0074745" rpy="0.0 -0.0 0.0"/>
       <mass value="0.42744"/>
-      <inertia ixx="0.00021055" ixy="3.1248e-10" ixz="-4.0813e-08" iyy="0.00010191" iyz="-4.0104e-07" izz="0.00021817"/>
+      <!-- <inertia ixx="0.00021055" ixy="3.1248e-10" ixz="-4.0813e-08" iyy="0.00010191" iyz="-4.0104e-07" izz="0.00021817"/> -->
+      <inertia ixx="6.32212e-04" ixy="4.40e-07" ixz="8.6305e-05" iyy="7.27448e-04" iyz="-1.4140e-05" izz="4.34901e-04"/>
     </inertial>
     <visual>
@@ -304,5 +323,6 @@
       <origin xyz="-0.16731 0.025056 -0.00016724" rpy="0.0 -0.0 0.0"/>
       <mass value="0.36482"/>
-      <inertia ixx="0.00016623" ixy="-3.3215e-07" ixz="-5.731e-09" iyy="0.00018621" iyz="-6.8029e-09" izz="0.00025293"/>
+      <!-- <inertia ixx="0.00016623" ixy="-3.3215e-07" ixz="-5.731e-09" iyy="0.00018621" iyz="-6.8029e-09" izz="0.00025293"/> -->
+      <inertia ixx="4.377329e-03" ixy="8.6412e-05" ixz="1.1901e-07" iyy="5.095606e-03" iyz="1.335e-06" izz="9.365966e-03"/>
     </inertial>
     <visual>
@@ -359,5 +379,6 @@
       <origin xyz="-3.541e-05 0.00191 0.0014323" rpy="0.0 -0.0 0.0"/>
       <mass value="0.32337"/>
-      <inertia ixx="0.0012194" ixy="2.2289e-07" ixz="-1.5989e-07" iyy="0.00099811" iyz="1.3306e-05" izz="0.0019906"/>
+      <!-- <inertia ixx="0.0012194" ixy="2.2289e-07" ixz="-1.5989e-07" iyy="0.00099811" iyz="1.3306e-05" izz="0.0019906"/> -->
+      <inertia ixx="2.041188e-03" ixy="-2.45e-07" ixz="3.31e-07" iyy="1.024308e-03" iyz="-1.287e-06" izz="2.793384e-03"/>
     </inertial>
     <visual>
@@ -369,8 +390,13 @@
   </link>
   <link name="thrust3">
-    <inertial>
-      <origin xyz="-2.7294e-06 -2.4294e-06 0.0039586" rpy="0.0 -0.0 0.0"/>
-      <mass value="0.010724"/>
-      <inertia ixx="1.6559e-05" ixy="-1.3706e-09" ixz="-2.9799e-11" iyy="1.6561e-05" iyz="1.1361e-11" izz="3.3082e-05"/>
+    <!-- <inertial> -->
+    <!--   <origin xyz="-2.7294e-06 -2.4294e-06 0.0039586" rpy="0.0 -0.0 0.0"/> -->
+    <!--   <mass value="0.010724"/> -->
+    <!--   <inertia ixx="1.6559e-05" ixy="-1.3706e-09" ixz="-2.9799e-11" iyy="1.6561e-05" iyz="1.1361e-11" izz="3.3082e-05"/> -->
+    <!-- </inertial> -->
+    <inertial>
+      <origin xyz="0 0 0" rpy="0 0 0"/>
+      <mass value="0.0001"/>
+      <inertia ixx="0.00001" ixy="0.0" ixz="0.0" iyy="0.00001" iyz="0.0" izz="0.00002"/>
     </inertial>
     <visual>
@@ -392,5 +418,6 @@
       <origin xyz="-0.036672 -2.1161e-05 0.0081671" rpy="0.0 -0.0 0.0"/>
       <mass value="0.31592"/>
-      <inertia ixx="5.7571e-05" ixy="6.2131e-09" ixz="8.7034e-08" iyy="9.2786e-05" iyz="-8.9132e-12" izz="7.7319e-05"/>
+      <!-- <inertia ixx="5.7571e-05" ixy="6.2131e-09" ixz="8.7034e-08" iyy="9.2786e-05" iyz="-8.9132e-12" izz="7.7319e-05"/> -->
+      <inertia ixx="4.69603e-04" ixy="1.87e-07" ixz="-3.7323e-05" iyy="5.56006e-04" iyz="-2.016e-05" izz="1.49828e-04"/>
     </inertial>
     <visual>
@@ -417,5 +444,6 @@
       <origin xyz="-0.056027 -0.0013733 0.0074745" rpy="0.0 -0.0 0.0"/>
       <mass value="0.42744"/>
-      <inertia ixx="0.00021055" ixy="3.1248e-10" ixz="-4.0813e-08" iyy="0.00010191" iyz="-4.0104e-07" izz="0.00021817"/>
+      <!-- <inertia ixx="0.00021055" ixy="3.1248e-10" ixz="-4.0813e-08" iyy="0.00010191" iyz="-4.0104e-07" izz="0.00021817"/> -->
+      <inertia ixx="6.32212e-04" ixy="4.40e-07" ixz="8.6305e-05" iyy="7.27448e-04" iyz="-1.4140e-05" izz="4.34901e-04"/>
     </inertial>
     <visual>
@@ -442,5 +470,6 @@
       <origin xyz="-0.16731 0.025056 -0.00016724" rpy="0.0 -0.0 0.0"/>
       <mass value="0.36482"/>
-      <inertia ixx="0.00016623" ixy="-3.3215e-07" ixz="-5.731e-09" iyy="0.00018621" iyz="-6.8029e-09" izz="0.00025293"/>
+      <!-- <inertia ixx="0.00016623" ixy="-3.3215e-07" ixz="-5.731e-09" iyy="0.00018621" iyz="-6.8029e-09" izz="0.00025293"/> -->
+      <inertia ixx="4.377329e-03" ixy="8.6412e-05" ixz="1.1901e-07" iyy="5.095606e-03" iyz="1.335e-06" izz="9.365966e-03"/>
     </inertial>
     <visual>
@@ -497,5 +526,6 @@
       <origin xyz="-3.541e-05 0.00191 0.0014323" rpy="0.0 -0.0 0.0"/>
       <mass value="0.32337"/>
-      <inertia ixx="0.0012194" ixy="2.2289e-07" ixz="-1.5989e-07" iyy="0.00099811" iyz="1.3306e-05" izz="0.0019906"/>
+      <!-- <inertia ixx="0.0012194" ixy="2.2289e-07" ixz="-1.5989e-07" iyy="0.00099811" iyz="1.3306e-05" izz="0.0019906"/> -->
+      <inertia ixx="2.041188e-03" ixy="-2.45e-07" ixz="3.31e-07" iyy="1.024308e-03" iyz="-1.287e-06" izz="2.793384e-03"/>
     </inertial>
     <visual>
@@ -507,8 +537,13 @@
   </link>
   <link name="thrust4">
-    <inertial>
-      <origin xyz="-2.7354e-06 -2.3382e-06 0.0039586" rpy="0.0 -0.0 0.0"/>
-      <mass value="0.010724"/>
-      <inertia ixx="1.6559e-05" ixy="-1.3583e-09" ixz="-2.999e-11" iyy="1.6561e-05" iyz="1.3027e-11" izz="3.3082e-05"/>
+    <!-- <inertial> -->
+    <!--   <origin xyz="-2.7354e-06 -2.3382e-06 0.0039586" rpy="0.0 -0.0 0.0"/> -->
+    <!--   <mass value="0.010724"/> -->
+    <!--   <inertia ixx="1.6559e-05" ixy="-1.3583e-09" ixz="-2.999e-11" iyy="1.6561e-05" iyz="1.3027e-11" izz="3.3082e-05"/> -->
+    <!-- </inertial> -->
+    <inertial>
+      <origin xyz="0 0 0" rpy="0 0 0"/>
+      <mass value="0.0001"/>
+      <inertia ixx="0.00001" ixy="0.0" ixz="0.0" iyy="0.00001" iyz="0.0" izz="0.00002"/>
     </inertial>
     <visual>
@@ -530,5 +565,6 @@
       <origin xyz="-0.036672 -2.1161e-05 0.0081671" rpy="0.0 -0.0 0.0"/>
       <mass value="0.31592"/>
-      <inertia ixx="5.7571e-05" ixy="6.2131e-09" ixz="8.7034e-08" iyy="9.2786e-05" iyz="-8.9133e-12" izz="7.7319e-05"/>
+      <!-- <inertia ixx="5.7571e-05" ixy="6.2131e-09" ixz="8.7034e-08" iyy="9.2786e-05" iyz="-8.9133e-12" izz="7.7319e-05"/> -->
+      <inertia ixx="4.69603e-04" ixy="1.87e-07" ixz="-3.7323e-05" iyy="5.56006e-04" iyz="-2.016e-05" izz="1.49828e-04"/>
     </inertial>
     <visual>
