Commit message: collisionを簡略化した。その結果imuのcalibがちゃんと行われ、rvizも正しく表示できるようになった。

File: robots/orochi_hx/urdf/orochi_hx_link.urdf.xacro (robot description, xacro)
@@ -17,9 +17,15 @@
           <origin xyz="0.0 0.0 0.0" rpy="0.0 -0.0 0.0"/>
         </visual>
-        <collision>
-          <geometry>
-            <mesh filename="package://orochi_hx/urdf/mesh/male_head_collision.stl"/>
-          </geometry>
-          <origin xyz="0.0 0.0 0.0" rpy="0.0 -0.0 0.0"/>
+        <collision name="male${self}_pipe_collision">
+          <geometry>
+            <box size="0.077 0.02 0.02"/>
+          </geometry>
+          <origin xyz="-0.0325 0 0" rpy="0.0 -0.0 0.0"/>
+        </collision>
+        <collision name="male${self}_leg_collision">
+          <geometry>
+            <box size="0.038 0.0525 0.07025"/>
+          </geometry>
+          <origin xyz="-0.051 0 -0.04512" rpy="0.0 -0.0 0.0"/>
         </collision>
       </xacro:if>
@@ -36,9 +42,15 @@
           <origin xyz="0.0 0.0 0.0" rpy="0.0 -0.0 0.0"/>
         </visual>
-        <collision>
-          <geometry>
-            <mesh filename="package://orochi_hx/urdf/mesh/male_collision.stl"/>
-          </geometry>
-          <origin xyz="0.0 0.0 0.0" rpy="0.0 -0.0 0.0"/>
+        <collision name="male${self}_pipe_collision">
+          <geometry>
+            <box size="0.077 0.02 0.02"/>
+          </geometry>
+          <origin xyz="-0.0325 0 0" rpy="0.0 -0.0 0.0"/>
+        </collision>
+        <collision name="male${self}_leg_collision">
+          <geometry>
+            <box size="0.038 0.0525 0.07025"/>
+          </geometry>
+          <origin xyz="-0.051 0 -0.04512" rpy="0.0 -0.0 0.0"/>
         </collision>
       </xacro:unless>
@@ -59,9 +71,27 @@
         <origin xyz="0.0 0.0 0.0" rpy="0.0 -0.0 0.0"/>
       </visual>
-      <collision>
-        <geometry>
-          <mesh filename="package://orochi_hx/urdf/mesh/body_collision.stl"/>
-        </geometry>
-        <origin xyz="0.0 0.0 0.0" rpy="0.0 -0.0 0.0"/>
+      <collision name="body${self}_long_pipe_left_collision">
+        <geometry>
+          <box size="0.166 0.01 0.03"/>
+        </geometry>
+        <origin xyz="0.0 0.142 0.0" rpy="0.0 -0.0 0.0"/>
+      </collision>
+      <collision name="body${self}_long_pipe_right_collision">
+        <geometry>
+          <box size="0.166 0.01 0.03"/>
+        </geometry>
+        <origin xyz="0.0 -0.142 0.0" rpy="0.0 -0.0 0.0"/>
+      </collision>
+      <collision name="body${self}_leg_left_collision">
+        <geometry>
+          <cylinder radius="0.0065" length="0.07025"/>
+        </geometry>
+        <origin xyz="0 0.1395 -0.05012" rpy="0 0 0"/>
+      </collision>
+      <collision name="body${self}_leg_right_collision">
+        <geometry>
+          <cylinder radius="0.0065" length="0.07025"/>
+        </geometry>
+        <origin xyz="0 -0.1395 -0.05012" rpy="0 0 0"/>
       </collision>
     </link>
@@ -81,9 +111,9 @@
         <origin xyz="0.0 0.0 0.0" rpy="0.0 -0.0 0.0"/>
       </visual>
-      <collision>
-        <geometry>
-          <mesh filename="package://orochi_hx/urdf/mesh/duct_collision.stl"/>
-        </geometry>
-        <origin xyz="0.0 0.0 0.0" rpy="0.0 -0.0 0.0"/>
+      <collision name="duct${self}_duct_collision">
+        <geometry>
+          <cylinder radius="0.1175" length="0.08"/>
+        </geometry>
+        <origin xyz="0.0 0.0 0.01" rpy="0.0 -0.0 0.0"/>
       </collision>
     </link>
@@ -104,9 +134,15 @@
           <origin xyz="0.0 0.0 0.0" rpy="0.0 -0.0 0.0"/>
         </visual>
-        <collision>
-          <geometry>
-            <mesh filename="package://orochi_hx/urdf/mesh/female_with_circuits_collision.stl"/>
-          </geometry>
-          <origin xyz="0.0 0.0 0.0" rpy="0.0 -0.0 0.0"/>
+        <collision name="female${self}_pipe_collision">
+          <geometry>
+            <box size="0.079 0.02 0.02"/>
+          </geometry>
+          <origin xyz="0.05903 0 0" rpy="0.0 -0.0 0.0"/>
+        </collision>
+        <collision name="female${self}_leg_collision">
+          <geometry>
+            <box size="0.038 0.0525 0.07025"/>
+          </geometry>
+          <origin xyz="0.07803 0 -0.05012" rpy="0.0 -0.0 0.0"/>
         </collision>
       </xacro:if>

Commit message: collisionの変更をしきれていなかった。シミュレーションが早くなった。

File: robots/orochi_hx/urdf/orochi_hx_link.urdf.xacro (robot description, xacro)
@@ -159,9 +159,15 @@
           <origin xyz="0.0 0.0 0.0" rpy="0.0 -0.0 0.0"/>
         </visual>
-        <collision>
-          <geometry>
-            <mesh filename="package://orochi_hx/urdf/mesh/female_collision.stl"/>
-          </geometry>
-          <origin xyz="0.0 0.0 0.0" rpy="0.0 -0.0 0.0"/>
+        <collision name="female${self}_pipe_collision">
+          <geometry>
+            <box size="0.079 0.02 0.02"/>
+          </geometry>
+          <origin xyz="0.05903 0 0" rpy="0.0 -0.0 0.0"/>
+        </collision>
+        <collision name="female${self}_leg_collision">
+          <geometry>
+            <box size="0.038 0.0525 0.07025"/>
+          </geometry>
+          <origin xyz="0.07803 0 -0.05012" rpy="0.0 -0.0 0.0"/>
         </collision>
       </xacro:unless>
@@ -194,10 +200,10 @@
         <origin xyz="0.0 0.0 0.0" rpy="0.0 -0.0 0.0"/>
       </visual>
-      <collision>
-        <geometry>
-          <mesh filename="package://orochi_hx/urdf/mesh/thrust_collision.stl"/>
-        </geometry>
-        <origin xyz="0.0 0.0 0.0" rpy="0.0 -0.0 0.0"/>
-      </collision>
+      <!-- <collision> -->
+      <!--   <geometry> -->
+      <!--     <mesh filename="package://orochi_hx/urdf/mesh/thrust_collision.stl"/> -->
+      <!--   </geometry> -->
+      <!--   <origin xyz="0.0 0.0 0.0" rpy="0.0 -0.0 0.0"/> -->
+      <!-- </collision> -->
     </link>
     <!-- <xacro:friction link="thrust${self}"/> -->

Commit message: urdfファイルの更新(revolute担っていなかったところを適用した)

File: robots/orochi_hx/urdf/orochi_hx_link.urdf.xacro (robot description, xacro)
@@ -277,5 +277,5 @@
     <xacro:implicit_damper joint="female_roll${self}"/>
     <xacro:unless value="${self == links}">
-      <joint name="joint_yaw${self}" type="continuous">
+      <joint name="joint_yaw${self}" type="revolute">
         <limit effort="10.0" lower="${-pi/2}" upper="${pi/2}" velocity="0.5"/>
         <!-- <limit effort="10.0" lower="${-pi/2}" upper="${pi/2}" velocity="0.1"/> -->
