Commit message: gazeboで一点に集まってしまう問題の解決。(damping_factorをimplicitにし、inertial paramをstl版に変更した)

File: robots/orochi_hx/urdf/orochi_hx_common.xacro (robot description, xacro)
@@ -27,4 +27,5 @@
     </gazebo>
   </xacro:macro>
+  <!-- damping factor -->
   <xacro:macro name="damping_factor" params="link">
     <gazebo reference="${link}">
@@ -32,3 +33,9 @@
     </gazebo>
   </xacro:macro>
+  <!-- implicit damper -->
+  <xacro:macro name="implicit_damper" params="joint">
+    <gazebo reference="${joint}">
+      <implicitSpringDamper>true</implicitSpringDamper>
+    </gazebo>
+  </xacro:macro>
 </robot>

File: robots/orochi_hx/urdf/orochi_hx_link.urdf.xacro (robot description, xacro)
@@ -7,7 +7,7 @@
       <xacro:if value="${self == 1}">
         <inertial>
-          <origin xyz="-0.052739878482681 -9.34675991357908e-07 -0.0296530174438008" rpy="0.0 -0.0 0.0"/>
-          <mass value="0.232368340978789"/>
-          <inertia ixx="0.000189201405336057" ixy="5.52592371497219e-09" ixz="3.65224196392575e-05" iyy="0.000272447160085503" iyz="-6.69151656946131e-10" izz="0.000168362228995049"/>
+          <origin xyz="-0.052739878482681 -9.34675991357908E-07 -0.0296530174438008" rpy="0 0 0" />
+          <mass value="0.232368340978789" />
+          <inertia ixx="0.000189201405336057" ixy="-5.52592371497092E-09" ixz="-3.65224196392574E-05" iyy="0.000272447160085503" iyz="6.69151656946078E-10" izz="0.000168362228995049" />
         </inertial>
         <visual>
@@ -26,7 +26,7 @@
       <xacro:unless value="${self == 1}">
         <inertial>
-          <origin xyz="0.480848878478817 -6.37525632024318e-07 -0.00526321596246022" rpy="0.0 -0.0 0.0"/>
-          <mass value="0.340677045513285"/>
-          <inertia ixx="0.000657095261464978" ixy="6.19678576389826e-09" ixz="8.97340693867749e-05" iyy="0.000757386523911567" iyz="4.62802062269456e-09" izz="0.000209861587892199"/>
+          <origin xyz="-0.0496511215211811 -6.37525642459786E-07 -0.00526321596244171" rpy="0 0 0" />
+          <mass value="0.340677045513285" />
+          <inertia ixx="0.000657095261464978" ixy="-6.19678576389833E-09" ixz="-8.97340693867749E-05" iyy="0.000757386523911568" iyz="-4.6280206226932E-09" izz="0.000209861587892199" />
         </inertial>
         <visual>
@@ -49,7 +49,7 @@
     <link name="body${self}">
       <inertial>
-        <origin xyz="0.249646267950928 0.0246488631309276 -0.00232944891667237" rpy="0.0 -0.0 0.0"/>
-        <mass value="0.419895456587595"/>
-        <inertia ixx="0.00520647615398925" ixy="-0.000107815705486367" ixz="-1.81339714467847e-06" iyy="0.00514529649185074" iyz="2.39989744251452e-05" izz="0.010151021448606"/>
+        <origin xyz="-0.00185373204907097 0.0246488631309219 -0.00232944891665445" rpy="0 0 0" />
+        <mass value="0.419895456587595" />
+        <inertia ixx="0.00520647615398925" ixy="0.000107815705486368" ixz="1.81339714467847E-06" iyy="0.00514529649185074" iyz="-2.39989744251452E-05" izz="0.010151021448606" />
       </inertial>
       <visual>
@@ -71,7 +71,7 @@
     <link name="duct${self}">
       <inertial>
-        <origin xyz="0.251457476616615 -0.00142751192883745 0.0011709194386648" rpy="0.0 -0.0 0.0"/>
-        <mass value="0.351486633634277"/>
-        <inertia ixx="0.0020630707445772" ixy="-2.92498532740653e-07" ixz="3.28976580216749e-07" iyy="0.00102307853147382" iyz="1.58803650253004e-07" izz="0.00281360888889416"/>
+        <origin xyz="-4.25233833842298E-05 -0.00142751192883604 0.00117091943866951" rpy="0 0 0" />
+        <mass value="0.351486633634277" />
+        <inertia ixx="0.0020630707445772" ixy="2.92498532740654E-07" ixz="-3.28976580216749E-07" iyy="0.00102307853147382" iyz="-1.58803650252997E-07" izz="0.00281360888889416" />
       </inertial>
       <visual>
@@ -94,7 +94,7 @@
       <xacro:if value="${self == 2}">
         <inertial>
-          <origin xyz="1.12698918290577 0.00619207162129304 -0.0202466021464508" rpy="0.0 -0.0 0.0"/>
-          <mass value="0.362731408934528"/>
-          <inertia ixx="0.000436668316629998" ixy="-8.91149536419333e-06" ixz="-0.000166184432843873" iyy="0.000716425694126863" iyz="8.2600244063983e-06" izz="0.000482080031496602"/>
+          <origin xyz="0.0659635829057773 0.00619207162128235 -0.0202466021464323" rpy="0 0 0" />
+          <mass value="0.362731408934528" />
+          <inertia ixx="0.000436668316629998" ixy="8.91149536419332E-06" ixz="0.000166184432843873" iyy="0.000716425694126863" iyz="-8.2600244063983E-06" izz="0.000482080031496602" />
         </inertial>
         <visual>
@@ -113,7 +113,7 @@
       <xacro:unless value="${self == 2}">
         <inertial>
-          <origin xyz="0.597343994892686 2.04473894948366e-05 -0.0246395348050693" rpy="0.0 -0.0 0.0"/>
-          <mass value="0.264982417970611"/>
-          <inertia ixx="0.000287291406649856" ixy="-3.80521104155563e-07" ixz="-0.000168019190894103" iyy="0.000596449506923116" iyz="3.358784385771e-07" izz="0.00040264407172139"/>
+          <origin xyz="0.0668183948926887 2.04473894828118E-05 -0.0246395348050516" rpy="0 0 0" />
+          <mass value="0.264982417970611" />
+          <inertia ixx="0.000287291406649856" ixy="3.80521104155564E-07" ixz="0.000168019190894103" iyy="0.000596449506923116" iyz="-3.35878438577101E-07" izz="0.00040264407172139" />
         </inertial>
         <visual>
@@ -212,4 +212,5 @@
       <dynamics damping="0.9" friction="0.05"/>
     </joint>
+    <xacro:implicit_damper joint="male_roll${self}"/>
     <joint name="gimbal_pitch${self}" type="revolute">
       <limit effort="1.5" lower="${-pi}" upper="${pi}" velocity="12.5"/>
@@ -221,4 +222,5 @@
       <dynamics damping="0.1" friction="0.0"/>
     </joint>
+    <xacro:implicit_damper joint="gimbal_pitch${self}"/>
     <joint name="female_roll${self}" type="revolute">
       <limit effort="5.0" lower="${-pi}" upper="${pi}" velocity="1.0"/>
@@ -231,4 +233,5 @@
       <dynamics damping="0.9" friction="0.05"/>
     </joint>
+    <xacro:implicit_damper joint="female_roll${self}"/>
     <xacro:unless value="${self == links}">
       <joint name="joint_yaw${self}" type="continuous">
@@ -243,4 +246,5 @@
         <dynamics damping="0.9" friction="0.05"/>
       </joint>
+      <xacro:implicit_damper joint="joint_yaw${self}"/>
     </xacro:unless>
     <xacro:if value="${self == 1}">

Commit message: 推力をat2814に合わせるのと同時にurdfのmax_forceも更新

File: robots/orochi_hx/urdf/orochi_hx_common.xacro (robot description, xacro)
@@ -18,5 +18,5 @@
   <!-- dynamics -->
   <m_f_rate value="-0.0172" /> <!-- drug torque rate -->
-  <xacro:property name="max_force" value="20.0" /> <!-- [N] -->
+  <xacro:property name="max_force" value="26.5" /> <!-- [N] -->
   <xacro:property name="min_force" value="1.0" /> <!-- [N] -->
     <!-- friction -->
